Commit message: fixed motor throttle equation

File: robot_description/urdf/quad.xacro (robot description, xacro)
@@ -22,9 +22,9 @@
     <inertial>
       <origin xyz="0 0 0" rpy="0 0 0"/>
-      <mass value="0.755"/>
+      <mass value="1.176"/>
       <inertia
-        ixx="0.005571050413" ixy="0.0" ixz="0.0"
-        iyy="0.005571050413" iyz="0.0"
-        izz="0.01050537595"/>
+        ixx="0.009773" ixy="0.0" ixz="0.0"
+        iyy="0.009773" iyz="0.0"
+        izz="0.01749"/>
     </inertial>
     <origin xyz="0 0 0" rpy="0 0 0" />

Commit message: some of the print variable removed
moved print statement to publisher for drone_variable msg

File: robot_description/urdf/quad.xacro (robot description, xacro)
@@ -22,5 +22,5 @@
     <inertial>
       <origin xyz="0 0 0" rpy="0 0 0"/>
-      <mass value="1.176"/>
+      <mass value="1.4"/>
       <inertia
         ixx="0.009773" ixy="0.0" ixz="0.0"
